Commit message: tiago urdf description compatible with ros2 and gazebo sim 8.8

File: urdf/tiago_from_our_robot.urdf (robot description, URDF)
Before this commit: robot tiago_dual, 102 links, 101 joints
Joints:
- joint gripper_left_left_inner_finger_joint: limit lower=-0.8757 upper=0 effort=0.1 velocity=2 -> lower=-0.8757 upper=0 effort=100.0 velocity=2
- joint gripper_left_left_inner_knuckle_joint: limit lower=0 upper=0.8757 effort=0.1 velocity=2 -> lower=0 upper=0.8757 effort=100.0 velocity=2
- joint gripper_left_right_inner_finger_joint: limit lower=-0.8757 upper=0 effort=0.1 velocity=2 -> lower=-0.8757 upper=0 effort=100.0 velocity=2
- joint gripper_left_right_inner_knuckle_joint: limit lower=0 upper=0.8757 effort=0.1 velocity=2 -> lower=0 upper=0.8757 effort=100.0 velocity=2
- joint gripper_left_right_outer_knuckle_joint: limit lower=0 upper=0.81 effort=0.1 velocity=2 -> lower=0 upper=0.81 effort=100.0 velocity=2
- joint gripper_right_left_inner_finger_joint: limit lower=-0.8757 upper=0 effort=0.1 velocity=2 -> lower=-0.8757 upper=0 effort=100.0 velocity=2
- joint gripper_right_left_inner_knuckle_joint: limit lower=0 upper=0.8757 effort=0.1 velocity=2 -> lower=0 upper=0.8757 effort=100.0 velocity=2
- joint gripper_right_right_inner_finger_joint: limit lower=-0.8757 upper=0 effort=0.1 velocity=2 -> lower=-0.8757 upper=0 effort=100.0 velocity=2
- joint gripper_right_right_inner_knuckle_joint: limit lower=0 upper=0.8757 effort=0.1 velocity=2 -> lower=0 upper=0.8757 effort=100.0 velocity=2
- joint gripper_right_right_outer_knuckle_joint: limit lower=0 upper=0.81 effort=0.1 velocity=2 -> lower=0 upper=0.81 effort=100.0 velocity=2
